File: eagle/PicKit2Clone.brd (EAGLE design)
At the start: 100 x 80 mm, 22 parts, among them IC1 PIC18F2550_28DIP, Q1 BC548, Q2 BC548, Q3 BC548, Q4 BC558A, Q5 BC548

Commit message: Esquematico terminado
Parts:
- added BUSSY, POWER: (no value), led:LED5MM
- added C4, C5: 22p, rcl:C025-024X044
- added C6: 100n, rcl:C025-024X044
- added D3: 1N4148DO35-7, diode:DO35-7
- added D4: 1N5817-T, diode:DO41-7.6
- added ISCP: 2510-, con-3m:PAK100/2500-10
- added JP1: (no value), pinhead:1X01
- added Q6, Q7, Q8: BC558A, transistor-pnp:TO92-EBC
- added Q9: 20MHz, special:QS
- added R11, R21: 10K, resistor:0204/5
- added R12, R13, R14: 33, resistor:0204/5
- added R15, R16: 4K7, resistor:0204/5
- added R17, R18, R19: 10, resistor:0204/5
- added R20: 100K, resistor:0204/5
- added R22, R23: 330, resistor:0204/5
- added SEL_VCC: (no value), pinhead:1X03
- added SW: PVA1R, switch-misc:PVA1R
- added USB: PN61729-S, con-berg:PN61729-S
Connections:
- new net N$11: D4.C, SEL_VCC.3
- new net N$12: Q6.E, R12.1, R19.1
- new net N$13: Q7.E, R13.1, R18.1
- new net N$14: Q8.E, R14.1, R17.1
- new net N$15: ISCP.10, ISCP.9, R13.2, R15.2
- new net N$16: ISCP.7, ISCP.8, R14.2, R16.2
- new net N$17: ISCP.1, ISCP.2
- new net N$18: ISCP.3, ISCP.4
- new net N$19: ISCP.5, ISCP.6
- new net N$20: D3.C, Q6.B, Q7.B, Q8.B, R20.1
- new net N$21: JP1.1, R12.2
- new net N$22: BUSSY.A, R23.1
- new net N$23: POWER.A, R22.1
- net +5V_USB: now also C6.1, D4.A, R21.2, R22.2, USB.1
- net AUX: now also R19.2
- net D+: now also USB.3
- net D-: now also USB.2
- net GND: now also BUSSY.K, C4.2, C5.2, C6.2, POWER.K, Q6.C, Q7.C, Q8.C, R15.1, R16.1, R20.2, SW.1, SW.3, USB.4, USB.S1, USB.S2
- net ISCP_CLK: now also R18.2
- net ISCP_DAT: now also R17.2
- net LED_BUSSY: now also R23.2
- net OSC1: now also C5.1, Q9.1
- net OSC2: now also C4.1, Q9.2
- net SW: now also R21.1, SW.2, SW.4
- net VDD_3.3V: now also SEL_VCC.1
- net VDD_FB: now also R11.1
- net VDD_TGT: now also D3.A, R11.2, SEL_VCC.2

Commit message: PCB a revisar
Parts:
- R1, R11, R12, R13, R14, R15, R16, R17, R18, R19, R20, R22, R23, R3, R5, R6, R7: device resistor:0204/5 -> resistor:0204/7
- moved POWER 369.1 mm to (90.2, 43.2)
- moved R21 363.5 mm to (27.9, 43.2)
- moved R22 360.0 mm to (90.2, 38.1), turned to 180 degrees
- moved BUSSY 351.1 mm to (90.2, 12.7)
- moved SW 349.3 mm to (27.9, 36.8)
- moved R23 346.7 mm to (74.9, 12.7), turned to 180 degrees
- moved C6 339.6 mm to (68.6, 34.3)
- moved USB 319.0 mm to (90.2, 27.9), turned to 90 degrees
- moved Q9 314.8 mm to (64.8, 16.5)
- moved C4 307.0 mm to (67.3, 12.7)
- moved C5 306.9 mm to (61.0, 12.7), turned to 180 degrees
- moved SEL_VCC 289.1 mm to (19.1, 43.2), turned to 90 degrees
- moved R20 277.2 mm to (35.6, 30.5), turned to 180 degrees
- moved JP1 270.4 mm to (10.2, 30.5)
- moved D3 267.4 mm to (39.4, 24.1), turned to 270 degrees
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Connections:
- removed net N$17: ISCP.1, ISCP.2
- removed net N$18: ISCP.3, ISCP.4
- removed net N$19: ISCP.5, ISCP.6
- net GND: now also ISCP.5, ISCP.6
- net ISCP_VPP: now also ISCP.1, ISCP.2
- net VDD_TGT: now also ISCP.3, ISCP.4
Routing:
- net ISCP_VPP: track 0.00 -> 163.9 mm, vias 0 -> 2
- net N$1: track 0.00 -> 127.4 mm, vias 0 -> 1
- net N$3: track 0.00 -> 126.5 mm
- net +5V_USB: track 0.00 -> 83.8 mm
- net VDD_TGT: track 0.00 -> 79.3 mm, vias 0 -> 1
- net VDD_3.3V: track 0.00 -> 59.3 mm, vias 0 -> 1
- net SW: track 0.00 -> 39.6 mm
- net AUX: track 0.00 -> 38.1 mm
- net ISCP_DAT: track 0.00 -> 35.7 mm
- net ISCP_CLK: track 0.00 -> 31.4 mm
- net N$4: track 0.00 -> 29.5 mm
- net N$13: track 0.00 -> 27.6 mm
- net N$15: track 0.00 -> 24.2 mm
- net N$16: track 0.00 -> 22.4 mm
- net N$20: track 0.00 -> 20.1 mm
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- added copper zone on layer 16, net GND
Other:
- board size 100 x 80 mm -> 94.9 x 46.2 mm

Commit message: Single layer Done
Parts:
- R1: device resistor:0204/7 -> resistor:0207/10
- R11, R12, R13, R14, R15, R16, R17, R18, R19, R22, R23, R3, R5, R7: device resistor:0204/7 -> resistor:0204/5
- R20: value 100K -> 820; device resistor:0204/7 -> resistor:0204/5
- moved R3 48.2 mm to (87.6, 40.6), turned to 180 degrees
- moved D1 46.2 mm to (83.8, 34.3), turned to 270 degrees
- moved L1 44.5 mm to (79.4, 30.5)
- moved SEL_VCC 39.6 mm to (58.4, 39.4), turned to 180 degrees
- moved R21 30.5 mm to (52.7, 25.4)
- moved Q2 28.0 mm to (66.0, 36.8), turned to 270 degrees
- moved R7 27.5 mm to (72.4, 30.5), turned to 90 degrees
- moved R17 26.8 mm to (48.9, 10.2), turned to 0 degrees
- moved R19 24.7 mm to (48.9, 5.71), turned to 0 degrees
- moved R15 24.4 mm to (37.5, 15.2)
- moved R13 23.3 mm to (37.5, 13.3)
- moved R16 23.2 mm to (38.1, 24.1)
- moved ISCP 23.0 mm to (31.1, 28.6)
- moved R14 22.9 mm to (38.1, 22.2)
- moved JP1 22.7 mm to (28.6, 17.1)
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Connections:
- removed net GNU: IC1.19
- net GND: now also IC1.19
Routing:
- net N$1: track 127.4 -> 4.44 mm, vias 1 -> 0
- net N$3: track 126.5 -> 9.93 mm
- net VPP_FB: track 12.5 -> 115.7 mm, vias 1 -> 0
- net ISCP_VPP: track 163.9 -> 62.2 mm, vias 2 -> 0
- net VDD_3.3V: track 59.3 -> 17.8 mm, vias 1 -> 0
- net VDD_TGT: track 79.3 -> 111.1 mm, vias 1 -> 0
- net +5V_USB: track 83.8 -> 56.2 mm
- net ISCP_DAT: track 35.7 -> 8.25 mm
- net AUX: track 38.1 -> 17.8 mm
- net N$4: track 29.5 -> 10.8 mm
- net SW: track 39.6 -> 20.9 mm
- net ISCP_CLK: track 31.4 -> 12.7 mm
- net N$13: track 27.6 -> 11.4 mm
- net N$14: track 6.35 -> 21.6 mm
- net N$16: track 22.4 -> 9.53 mm
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