File: eagle/PicKit2Clone.sch (EAGLE design)
At the start: 22 parts, among them IC1 PIC18F2550_28DIP, Q1 BC548, Q2 BC548, Q3 BC548, Q4 BC558A, Q5 BC548

Commit message: Esquematico terminado
Parts:
- added BUSSY, POWER: (no value), led:LED5MM
- added C4, C5: 22p, rcl:C-EU025-024X044
- added C6: 100n, rcl:C-EU025-024X044
- added D3: 1N4148DO35-7, diode:1N4148DO35-7
- added D4: 1N5817-T, diode:1N5817-T
- added ISCP: 2510-, con-3m:2510-
- added JP1: (no value), pinhead:PINHD-1X1
- added Q6, Q7, Q8: BC558A, transistor-pnp:BC558A
- added Q9: 20MHz, special:XTAL/S
- added R11, R21: 10K, resistor:R-EU_0204/5
- added R12, R13, R14: 33, resistor:R-EU_0204/5
- added R15, R16: 4K7, resistor:R-EU_0204/5
- added R17, R18, R19: 10, resistor:R-EU_0204/5
- added R20: 100K, resistor:R-EU_0204/5
- added R22, R23: 330, resistor:R-EU_0204/5
- added SEL_VCC: (no value), pinhead:PINHD-1X3
- added SW: PVA1R, switch-misc:PVA1R
- added USB: PN61729-S, con-berg:PN61729-S
Connections:
- new net N$11: D4.C, SEL_VCC.3
- new net N$12: Q6.E, R12.1, R19.1
- new net N$13: Q7.E, R13.1, R18.1
- new net N$14: Q8.E, R14.1, R17.1
- new net N$15: ISCP-10.KL, ISCP-9.KL, R13.2, R15.2
- new net N$16: ISCP-7.KL, ISCP-8.KL, R14.2, R16.2
- new net N$17: ISCP-1.KL, ISCP-2.KL
- new net N$18: ISCP-3.KL, ISCP-4.KL
- new net N$19: ISCP-5.KL, ISCP-6.KL
- new net N$20: D3.C, Q6.B, Q7.B, Q8.B, R20.1
- new net N$21: JP1.1, R12.2
- new net N$22: BUSSY.A, R23.1
- new net N$23: POWER.A, R22.1
- net +5V_USB: now also C6.1, D4.A, R21.2, R22.2, USB.1
- net AUX: now also R19.2
- net D+: now also USB.3
- net D-: now also USB.2
- net GND: now also BUSSY.C, C4.2, C5.2, C6.2, POWER.C, Q6.C, Q7.C, Q8.C, R15.1, R16.1, R20.2, SW1.S, SW2.S, USB.4, USB.S1, USB.S2
- net ISCP_CLK: now also R18.2
- net ISCP_DAT: now also R17.2
- net LED_BUSSY: now also R23.2
- net OSC1: now also C5.1, Q9.1
- net OSC2: now also C4.1, Q9.2
- net SW: now also R21.1, SW1.P, SW2.P
- net VDD_3.3V: now also SEL_VCC.1
- net VDD_FB: now also R11.1
- net VDD_TGT: now also D3.A, R11.2, SEL_VCC.2
Other:
- moved on the sheet: C1, C2, C3, D1, D2, IC1, L1, Q1, Q2, Q3, Q4, Q5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

Commit message: PCB a revisar
Parts:
- R1, R11, R12, R13, R14, R15, R16, R17, R18, R19, R20, R22, R23, R3, R5, R6, R7: device resistor:R-EU_0204/5 -> resistor:R-EU_0204/7
Connections:
- removed net N$17: ISCP-1.KL, ISCP-2.KL
- removed net N$18: ISCP-3.KL, ISCP-4.KL
- removed net N$19: ISCP-5.KL, ISCP-6.KL
- net GND: now also ISCP-5.KL, ISCP-6.KL
- net ISCP_VPP: now also ISCP-1.KL, ISCP-2.KL
- net VDD_TGT: now also ISCP-3.KL, ISCP-4.KL

Commit message: Single layer Done
Parts:
- R1: device resistor:R-EU_0204/7 -> resistor:R-EU_0207/10
- R11, R12, R13, R14, R15, R16, R17, R18, R19, R22, R23, R3, R5, R7: device resistor:R-EU_0204/7 -> resistor:R-EU_0204/5
- R20: value 100K -> 820; device resistor:R-EU_0204/7 -> resistor:R-EU_0204/5
Connections:
- removed net GNU: IC1.VSS@1
- net GND: now also IC1.VSS@1
Changed lines of the file:
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@@
 <?xml version="1.0" encoding="utf-8"?>
 <!DOCTYPE eagle SYSTEM "eagle.dtd">
-<eagle version="6.5.0">
+<eagle version="7.4.0">
 <drawing>
 <settings>
@@
 <part name="L1" library="rcl" deviceset="L-EU" device="0204/5" value="680uHy"/>
 <part name="D1" library="diode" deviceset="1N4148" device="DO35-7"/>
-<part name="R1" library="resistor" deviceset="R-EU_" device="0204/7" value="1K"/>
+<part name="R1" library="resistor" deviceset="R-EU_" device="0207/10" value="1K"/>
 <part name="R2" library="resistor" deviceset="R-EU_" device="0204/5" value="4K7"/>
-<part name="R3" library="resistor" deviceset="R-EU_" device="0204/7" value="2K7"/>
+<part name="R3" library="resistor" deviceset="R-EU_" device="0204/5" value="2K7"/>
 <part name="R4" library="resistor" deviceset="R-EU_" device="0204/5" value="100K"/>
 <part name="Q1" library="transistor-npn" deviceset="BC548*" device=""/>
 <part name="GND1" library="supply1" deviceset="GND" device=""/>
-<part name="R5" library="resistor" deviceset="R-EU_" device="0204/7" value="10K"/>
+<part name="R5" library="resistor" deviceset="R-EU_" device="0204/5" value="10K"/>
 <part name="GND2" library="supply1" deviceset="GND" device=""/>
 <part name="GND4" library="supply1" deviceset="GND" device=""/>
@@
 <part name="Q2" library="transistor-npn" deviceset="BC548*" device=""/>
 <part name="R6" library="resistor" deviceset="R-EU_" device="0204/7" value="10K"/>
-<part name="R7" library="resistor" deviceset="R-EU_" device="0204/7" value="10K"/>
+<part name="R7" library="resistor" deviceset="R-EU_" device="0204/5" value="10K"/>
 <part name="R8" library="resistor" deviceset="R-EU_" device="0204/5" value="10K"/>
 <part name="GND3" library="supply1" deviceset="GND" device=""/>
@@
 <part name="GND9" library="supply1" deviceset="GND" device=""/>
 <part name="D4" library="diode" deviceset="1N581*" device="" technology="7-T"/>
-<part name="R11" library="resistor" deviceset="R-EU_" device="0204/7" value="10K"/>
+<part name="R11" library="resistor" deviceset="R-EU_" device="0204/5" value="10K"/>
 <part name="ISCP" library="con-3m" deviceset="2510-" device=""/>
-<part name="R12" library="resistor" deviceset="R-EU_" device="0204/7" value="33"/>
-<part name="R13" library="resistor" deviceset="R-EU_" device="0204/7" value="33"/>
+<part name="R12" library="resistor" deviceset="R-EU_" device="0204/5" value="33"/>
+<part name="R13" library="resistor" deviceset="R-EU_" device="0204/5" value="33"/>
 <part name="Q7" library="transistor-pnp" deviceset="BC558*" device="" technology="A"/>
 <part name="Q6" library="transistor-pnp" deviceset="BC558*" device="" technology="A"/>
-<part name="R14" library="resistor" deviceset="R-EU_" device="0204/7" value="33"/>
+<part name="R14" library="resistor" deviceset="R-EU_" device="0204/5" value="33"/>
 <part name="Q8" library="transistor-pnp" deviceset="BC558*" device="" technology="A"/>
-<part name="R15" library="resistor" deviceset="R-EU_" device="0204/7" value="4K7"/>
-<part name="R16" library="resistor" deviceset="R-EU_" device="0204/7" value="4K7"/>
-<part name="R17" library="resistor" deviceset="R-EU_" device="0204/7" value="10"/>
+<part name="R15" library="resistor" deviceset="R-EU_" device="0204/5" value="4K7"/>
+<part name="R16" library="resistor" deviceset="R-EU_" device="0204/5" value="4K7"/>
+<part name="R17" library="resistor" deviceset="R-EU_" device="0204/5" value="10"/>
 <part name="GND10" library="supply1" deviceset="GND" device=""/>
 <part name="GND11" library="supply1" deviceset="GND" device=""/>
@@
 <part name="GND13" library="supply1" deviceset="GND" device=""/>
 <part name="GND14" library="supply1" deviceset="GND" device=""/>
-<part name="R19" library="resistor" deviceset="R-EU_" device="0204/7" value="10"/>
-<part name="R18" library="resistor" deviceset="R-EU_" device="0204/7" value="10"/>
+<part name="R19" library="resistor" deviceset="R-EU_" device="0204/5" value="10"/>
+<part name="R18" library="resistor" deviceset="R-EU_" device="0204/5" value="10"/>
 <part name="D3" library="diode" deviceset="1N4148" device="DO35-7"/>
-<part name="R20" library="resistor" deviceset="R-EU_" device="0204/7" value="100K"/>
+<part name="R20" library="resistor" deviceset="R-EU_" device="0204/5" value="820"/>
 <part name="GND15" library="supply1" deviceset="GND" device=""/>
 <part name="JP1" library="pinhead" deviceset="PINHD-1X1" device=""/>
@@
 <part name="GND20" library="supply1" deviceset="GND" device=""/>
 <part name="C6" library="rcl" deviceset="C-EU" device="025-024X044" value="100n"/>
-<part name="R22" library="resistor" deviceset="R-EU_" device="0204/7" value="330"/>
+<part name="R22" library="resistor" deviceset="R-EU_" device="0204/5" value="330"/>
 <part name="POWER" library="led" deviceset="LED" device="5MM"/>
 <part name="BUSSY" library="led" deviceset="LED" device="5MM"/>
-<part name="R23" library="resistor" deviceset="R-EU_" device="0204/7" value="330"/>
+<part name="R23" library="resistor" deviceset="R-EU_" device="0204/5" value="330"/>
 <part name="SW" library="switch-misc" deviceset="PVA1R" device=""/>
 <part name="GND21" library="supply1" deviceset="GND" device=""/>
@@
 <wire x1="86.36" y1="68.58" x2="93.98" y2="68.58" width="0.1524" layer="91"/>
 <label x="91.44" y="68.58" size="1.778" layer="95"/>
+<junction x="86.36" y="68.58"/>
+<junction x="83.82" y="68.58"/>
 </segment>
 <segment>
@@
 <junction x="193.04" y="147.32"/>
 </segment>
+<segment>
+<pinref part="IC1" gate="G$1" pin="VSS@1"/>
+<wire x1="53.34" y1="114.3" x2="60.96" y2="114.3" width="0.1524" layer="91"/>
+<label x="55.88" y="114.3" size="1.778" layer="95"/>
+</segment>
 </net>
 <net name="OSC1" class="0">
@@
 <wire x1="7.62" y1="66.04" x2="7.62" y2="73.66" width="0.1524" layer="91"/>
 <label x="7.62" y="73.66" size="1.778" layer="95" rot="R90"/>
+<junction x="7.62" y="66.04"/>
 </segment>
 </net>
@@
 <wire x1="17.78" y1="66.04" x2="17.78" y2="73.66" width="0.1524" layer="91"/>
 <label x="17.78" y="73.66" size="1.778" layer="95" rot="R90"/>
+<junction x="17.78" y="66.04"/>
 </segment>
 </net>
@@
 <wire x1="-35.56" y1="78.74" x2="-35.56" y2="86.36" width="0.1524" layer="91"/>
 <label x="-35.56" y="81.28" size="1.778" layer="95" rot="R90"/>
-</segment>
-</net>
-<net name="GNU" class="0">
-<segment>
-<pinref part="IC1" gate="G$1" pin="VSS@1"/>
-<wire x1="53.34" y1="114.3" x2="60.96" y2="114.3" width="0.1524" layer="91"/>
-<label x="55.88" y="114.3" size="1.778" layer="95"/>
 </segment>
 </net>
@@
 <wire x1="172.72" y1="12.7" x2="190.5" y2="12.7" width="0.1524" layer="91"/>
 <label x="177.8" y="12.7" size="1.778" layer="95"/>
+<junction x="172.72" y="12.7"/>
 </segment>
 <segment>
@@
 <wire x1="193.04" y1="165.1" x2="177.8" y2="165.1" width="0.1524" layer="91"/>
 <label x="175.26" y="165.1" size="1.778" layer="95"/>
+<junction x="193.04" y="165.1"/>
 </segment>
 </net>
@@
 <wire x1="190.5" y1="109.22" x2="180.34" y2="109.22" width="0.1524" layer="91"/>
 <junction x="180.34" y="109.22"/>
+<junction x="190.5" y="109.22"/>
 </segment>
 </net>
@@
 <wire x1="193.04" y1="83.82" x2="180.34" y2="83.82" width="0.1524" layer="91"/>
 <junction x="180.34" y="83.82"/>
-</segment>
-</net>
+<junction x="193.04" y="83.82"/>
+</segment>
+</net>
