File: eagle/PicKit2Clone2.sch (EAGLE design)
At the start: 51 parts, among them IC1 PIC18F2550_28DIP, Q1 BC548, Q2 BC548, Q3 BC548, Q4 BC558A, Q5 BC548, Q6 BC558A, Q7 BC558A, Q8 BC558A, Q9 20MHz

Commit message: mejora de 5x5
Parts:
- USB: value PN61729-S -> (none); device con-berg:PN61729-S -> con-berg:PN61729
Connections:
- net GND: no longer USB.S1, USB.S2
Changed lines of the file:
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@@
 <part name="JP1" library="pinhead" deviceset="PINHD-1X1" device=""/>
 <part name="SEL_VCC" library="pinhead" deviceset="PINHD-1X3" device=""/>
-<part name="USB" library="con-berg" deviceset="PN61729-S" device=""/>
+<part name="USB" library="con-berg" deviceset="PN61729" device=""/>
 <part name="C4" library="rcl" deviceset="C-EU" device="025-024X044" value="22p"/>
 <part name="C5" library="rcl" deviceset="C-EU" device="025-024X044" value="22p"/>
@@
 </segment>
 <segment>
-<pinref part="USB" gate="G$1" pin="S1"/>
-<pinref part="USB" gate="G$1" pin="S2"/>
-<wire x1="83.82" y1="68.58" x2="86.36" y2="68.58" width="0.1524" layer="91"/>
-<wire x1="86.36" y1="68.58" x2="93.98" y2="68.58" width="0.1524" layer="91"/>
-<label x="91.44" y="68.58" size="1.778" layer="95"/>
-<junction x="86.36" y="68.58"/>
-<junction x="83.82" y="68.58"/>
-</segment>
-<segment>

Commit message: cambios menores
Parts:
- D2: value 1N4728 -> 1N4731; device diode:1N4728 -> diode:ZENER-DIODEDO41Z10
- R11: value 10K -> 4K7
- R7: value 10K -> 100
Changed lines of the file:
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@@
 <?xml version="1.0" encoding="utf-8"?>
 <!DOCTYPE eagle SYSTEM "eagle.dtd">
-<eagle version="7.4.0">
+<eagle version="6.5.0">
 <drawing>
 <settings>
@@
 <part name="Q2" library="transistor-npn" deviceset="BC548*" device=""/>
 <part name="R6" library="resistor" deviceset="R-EU_" device="0204/7" value="10K"/>
-<part name="R7" library="resistor" deviceset="R-EU_" device="0204/5" value="10K"/>
+<part name="R7" library="resistor" deviceset="R-EU_" device="0204/5" value="100"/>
 <part name="R8" library="resistor" deviceset="R-EU_" device="0204/7" value="10K"/>
 <part name="GND3" library="supply1" deviceset="GND" device=""/>
@@
 <part name="C2" library="rcl" deviceset="CPOL-EU" device="E1.8-4" value="1uF"/>
 <part name="GND8" library="supply1" deviceset="GND" device=""/>
-<part name="D2" library="diode" deviceset="1N4728" device=""/>
+<part name="D2" library="diode" deviceset="ZENER-DIODE" device="DO41Z10" value="1N4731"/>
 <part name="GND9" library="supply1" deviceset="GND" device=""/>
 <part name="D4" library="diode" deviceset="1N581*" device="" technology="7-T"/>
-<part name="R11" library="resistor" deviceset="R-EU_" device="0204/5" value="10K"/>
+<part name="R11" library="resistor" deviceset="R-EU_" device="0204/5" value="4K7"/>
 <part name="ISCP" library="con-3m" deviceset="2510-" device=""/>
 <part name="R12" library="resistor" deviceset="R-EU_" device="0204/5" value="33"/>
@@
 <instance part="C2" gate="G$1" x="-30.48" y="104.14" rot="R270"/>
 <instance part="GND8" gate="1" x="-40.64" y="101.6"/>
-<instance part="D2" gate="1" x="30.48" y="2.54" rot="R90"/>
+<instance part="D2" gate="G$1" x="30.48" y="2.54" rot="R90"/>
 <instance part="GND9" gate="1" x="30.48" y="-2.54"/>
 <instance part="D4" gate="G$1" x="0" y="17.78" rot="R180"/>
@@
 </segment>
 <segment>
-<pinref part="D2" gate="1" pin="A"/>
+<pinref part="D2" gate="G$1" pin="A"/>
 <pinref part="GND9" gate="1" pin="GND"/>
 </segment>
@@
 <pinref part="Q5" gate="G$1" pin="B"/>
 <wire x1="43.18" y1="12.7" x2="30.48" y2="12.7" width="0.1524" layer="91"/>
-<pinref part="D2" gate="1" pin="C"/>
+<pinref part="D2" gate="G$1" pin="C"/>
 <wire x1="30.48" y1="5.08" x2="30.48" y2="12.7" width="0.1524" layer="91"/>
 <junction x="30.48" y="12.7"/>
